File: thin-key.kicad_pcb (KiCad board)
At the start: 2 copper layers, 77 x 44 mm, 9 parts, among them SW1 SW_PUSH, SW2 SW_PUSH, SW3 SW_PUSH, SW4 SW_PUSH, U1 Pico

Commit message: Use single layer
Routing:
- net col0: track 19.1 -> 47.3 mm
- net col1: track 19.0 -> 39.0 mm
- net Net-(D4-Pad2): track 45.7 -> 46.8 mm
- net row1: track 36.2 -> 37.0 mm, vias 1 -> 0
- net Net-(D1-Pad2): track 24.1 -> 24.2 mm, vias 1 -> 0
Changed lines of the file:
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@@
   (segment (start 91.44 102.49) (end 115.19 102.49) (width 0.25) (layer "F.Cu") (net 1))
   (segment (start 88.9 102.49) (end 91.44 102.49) (width 0.25) (layer "F.Cu") (net 1))
+  (segment (start 87.25 101.6) (end 116.84 101.6) (width 0.25) (layer "F.Cu") (net 2))
+  (segment (start 116.84 101.6) (end 119.38 104.14) (width 0.25) (layer "F.Cu") (net 2))
+  (segment (start 86.36 102.49) (end 87.25 101.6) (width 0.25) (layer "F.Cu") (net 2))
   (segment (start 83.82 102.49) (end 86.36 102.49) (width 0.25) (layer "F.Cu") (net 2))
-  (via (at 86.36 102.49) (size 0.8) (drill 0.4) (layers "F.Cu" "B.Cu") (net 2))
-  (segment (start 86.36 102.49) (end 117.73 102.49) (width 0.25) (layer "B.Cu") (net 2))
-  (segment (start 117.73 102.49) (end 119.38 104.14) (width 0.25) (layer "B.Cu") (net 2))
-  (segment (start 107.499992 114.299836) (end 88.449992 114.299836) (width 0.25) (layer "F.Cu") (net 3))
+  (segment (start 109.22 104.14) (end 109.22 112.579828) (width 0.25) (layer "F.Cu") (net 3))
+  (segment (start 105.409836 114.299836) (end 107.499992 114.299836) (width 0.25) (layer "F.Cu") (net 3))
+  (segment (start 109.22 112.579828) (end 107.499992 114.299836) (width 0.25) (layer "F.Cu") (net 3))
+  (segment (start 96.125 105.015) (end 105.409836 114.299836) (width 0.25) (layer "F.Cu") (net 3))
+  (segment (start 88.449992 110.900696) (end 85.435 107.885704) (width 0.25) (layer "F.Cu") (net 3))
+  (segment (start 85.435 107.885704) (end 85.435 105.015) (width 0.25) (layer "F.Cu") (net 3))
+  (segment (start 85.435 105.015) (end 96.125 105.015) (width 0.25) (layer "F.Cu") (net 3))
+  (segment (start 88.449992 114.299836) (end 88.449992 110.900696) (width 0.25) (layer "F.Cu") (net 3))
+  (segment (start 111.76 104.14) (end 111.76 105.75) (width 0.25) (layer "F.Cu") (net 4))
   (segment (start 126.549992 114.299836) (end 145.599992 114.299836) (width 0.25) (layer "F.Cu") (net 4))
-  (via (at 88.9 105.918) (size 0.8) (drill 0.4) (layers "F.Cu" "B.Cu") (net 40))
-  (segment (start 102.181836 119.199836) (end 107.499992 119.199836) (width 0.25) (layer "B.Cu") (net 40))
-  (segment (start 88.9 105.918) (end 102.181836 119.199836) (width 0.25) (layer "B.Cu") (net 40))
+  (segment (start 111.76 105.75) (end 120.309836 114.299836) (width 0.25) (layer "F.Cu") (net 4))
+  (segment (start 120.309836 114.299836) (end 126.549992 114.299836) (width 0.25) (layer "F.Cu") (net 4))
+  (segment (start 107.499992 119.199836) (end 102.309836 119.199836) (width 0.25) (layer "F.Cu") (net 40))
+  (segment (start 102.309836 119.199836) (end 88.9 105.79) (width 0.25) (layer "F.Cu") (net 40))
   (segment (start 83.82 105.79) (end 83.82 114.569844) (width 0.25) (layer "F.Cu") (net 41))
   (segment (start 83.82 114.569844) (end 88.449992 119.199836) (width 0.25) (layer "F.Cu") (net 41))
-  (segment (start 117.774367 107.114511) (end 126.335336 115.67548) (width 0.25) (layer "F.Cu") (net 42))
-  (segment (start 91.44 105.79) (end 92.764511 107.114511) (width 0.25) (layer "F.Cu") (net 42))
-  (segment (start 92.764511 107.114511) (end 117.774367 107.114511) (width 0.25) (layer "F.Cu") (net 42))
-  (segment (start 126.335336 115.67548) (end 142.075636 115.67548) (width 0.25) (layer "F.Cu") (net 42))
-  (segment (start 142.075636 115.67548) (end 145.599992 119.199836) (width 0.25) (layer "F.Cu") (net 42))
-  (segment (start 120.525481 113.175325) (end 126.549992 119.199836) (width 0.25) (layer "F.Cu") (net 43))
-  (segment (start 86.36 105.79) (end 93.745325 113.175325) (width 0.25) (layer "F.Cu") (net 43))
-  (segment (start 93.745325 113.175325) (end 120.525481 113.175325) (width 0.25) (layer "F.Cu") (net 43))
+  (segment (start 101.325 115.675) (end 142.075156 115.675) (width 0.25) (layer "F.Cu") (net 42))
+  (segment (start 91.44 105.79) (end 101.325 115.675) (width 0.25) (layer "F.Cu") (net 42))
+  (segment (start 142.075156 115.675) (end 145.599992 119.199836) (width 0.25) (layer "F.Cu") (net 42))
+  (segment (start 86.36 105.79) (end 101.095 120.525) (width 0.25) (layer "F.Cu") (net 43))
+  (segment (start 101.095 120.525) (end 125.224828 120.525) (width 0.25) (layer "F.Cu") (net 43))
+  (segment (start 125.224828 120.525) (end 126.549992 119.199836) (width 0.25) (layer "F.Cu") (net 43))
 )
