File: thin-key.kicad_pcb (KiCad board)
At the start: 2 copper layers, 77 x 44 mm, 9 parts, among them SW1 SW_PUSH, SW2 SW_PUSH, SW3 SW_PUSH, SW4 SW_PUSH, U1 Pico

Commit message: Add jlcjlcjlcjlc
Parts:
- moved D1 5.08 mm to (88.9, 104.1)
- moved D3 5.08 mm to (91.4, 104.1)
Routing:
- net row0: track 23.5 -> 28.6 mm
- net Net-(D1-Pad2): track 19.0 -> 24.1 mm
- net Net-(D3-Pad2): track 54.6 -> 59.7 mm
Other:
- board text added: "JLCJLCJLCJLC"
Changed lines of the file:
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@@
       (outputformat 1)
       (mirror false)
-      (drillshape 1)
+      (drillshape 0)
       (scaleselection 1)
-      (outputdirectory "")
+      (outputdirectory "dist/")
     )
   )
@@
   (net 47 "unconnected-(U1-Pad5)")
   (footprint "Diode_SMD:D_SOD-123" (layer "F.Cu")
-    (at 93.98 104.14 -90)
+    (at 88.9 104.14 -90)
     (descr "SOD-123")
     (tags "SOD-123")
@@
     (property "Sheetname" "")
     (attr smd)
-    (fp_text reference "D1" (at -0.45 -4.7 90) (layer "F.SilkS")
+    (fp_text reference "D1" (at -3.556 0 90) (layer "F.SilkS")
       (effects (font (size 1 1) (thickness 0.15)))
     )
     (fp_text value "1N4148W" (at 0 2.1 90) (layer "F.Fab")
-      (effects (font (size 1 1) (thickness 0.15)))
-    )
-    (fp_text user "${REFERENCE}" (at -0.45 -4.7 90) (layer "F.Fab")
       (effects (font (size 1 1) (thickness 0.15)))
     )
@@
     (property "Sheetname" "")
     (attr smd)
-    (fp_text reference "D2" (at 0 -2 90) (layer "F.SilkS")
+    (fp_text reference "D2" (at -3.556 0 90) (layer "F.SilkS")
       (effects (font (size 1 1) (thickness 0.15)))
     )
@@
   )
   (footprint "Diode_SMD:D_SOD-123" (layer "F.Cu")
-    (at 96.52 104.14 -90)
+    (at 91.44 104.14 -90)
     (descr "SOD-123")
     (tags "SOD-123")
@@
     (property "Sheetname" "")
     (attr smd)
-    (fp_text reference "D3" (at 2.55 -1.985 90) (layer "F.SilkS")
+    (fp_text reference "D3" (at -3.556 0 90) (layer "F.SilkS")
       (effects (font (size 1 1) (thickness 0.15)))
     )
@@
     (property "Sheetname" "")
     (attr smd)
-    (fp_text reference "D4" (at 0 -2 90) (layer "F.SilkS")
+    (fp_text reference "D4" (at -3.556 0 90) (layer "F.SilkS")
       (effects (font (size 1 1) (thickness 0.15)))
     )
@@
   (gr_line (start 82 83) (end 82 127) (layer "Edge.Cuts") (width 0.1))
   (gr_line (start 159 127) (end 159 83) (layer "Edge.Cuts") (width 0.1))
+  (gr_text "JLCJLCJLCJLC" (at 151 90) (layer "F.SilkS")
+    (effects (font (size 1 1) (thickness 0.15)))
+  )
   (segment (start 115.19 102.49) (end 116.84 104.14) (width 0.25) (layer "F.Cu") (net 1))
-  (segment (start 93.98 102.49) (end 96.52 102.49) (width 0.25) (layer "F.Cu") (net 1))
-  (segment (start 96.52 102.49) (end 115.19 102.49) (width 0.25) (layer "F.Cu") (net 1))
+  (segment (start 91.44 102.49) (end 115.19 102.49) (width 0.25) (layer "F.Cu") (net 1))
+  (segment (start 88.9 102.49) (end 91.44 102.49) (width 0.25) (layer "F.Cu") (net 1))
   (segment (start 83.82 102.49) (end 86.36 102.49) (width 0.25) (layer "F.Cu") (net 2))
   (via (at 86.36 102.49) (size 0.8) (drill 0.4) (layers "F.Cu" "B.Cu") (net 2))
@@
   (segment (start 107.499992 114.299836) (end 88.449992 114.299836) (width 0.25) (layer "F.Cu") (net 3))
   (segment (start 126.549992 114.299836) (end 145.599992 114.299836) (width 0.25) (layer "F.Cu") (net 4))
-  (via (at 93.98 105.918) (size 0.8) (drill 0.4) (layers "F.Cu" "B.Cu") (net 40))
-  (segment (start 93.98 105.918) (end 94.218156 105.918) (width 0.25) (layer "B.Cu") (net 40))
-  (segment (start 94.218156 105.918) (end 107.499992 119.199836) (width 0.25) (layer "B.Cu") (net 40))
+  (via (at 88.9 105.918) (size 0.8) (drill 0.4) (layers "F.Cu" "B.Cu") (net 40))
+  (segment (start 102.181836 119.199836) (end 107.499992 119.199836) (width 0.25) (layer "B.Cu") (net 40))
+  (segment (start 88.9 105.918) (end 102.181836 119.199836) (width 0.25) (layer "B.Cu") (net 40))
   (segment (start 83.82 105.79) (end 83.82 114.569844) (width 0.25) (layer "F.Cu") (net 41))
   (segment (start 83.82 114.569844) (end 88.449992 119.199836) (width 0.25) (layer "F.Cu") (net 41))
-  (segment (start 96.52 105.79) (end 103.454357 112.724357) (width 0.25) (layer "F.Cu") (net 42))
-  (segment (start 123.384213 112.724357) (end 126.229856 115.57) (width 0.25) (layer "F.Cu") (net 42))
-  (segment (start 141.970156 115.57) (end 145.599992 119.199836) (width 0.25) (layer "F.Cu") (net 42))
-  (segment (start 126.229856 115.57) (end 141.970156 115.57) (width 0.25) (layer "F.Cu") (net 42))
-  (segment (start 103.454357 112.724357) (end 123.384213 112.724357) (width 0.25) (layer "F.Cu") (net 42))
+  (segment (start 117.774367 107.114511) (end 126.335336 115.67548) (width 0.25) (layer "F.Cu") (net 42))
+  (segment (start 91.44 105.79) (end 92.764511 107.114511) (width 0.25) (layer "F.Cu") (net 42))
+  (segment (start 92.764511 107.114511) (end 117.774367 107.114511) (width 0.25) (layer "F.Cu") (net 42))
+  (segment (start 126.335336 115.67548) (end 142.075636 115.67548) (width 0.25) (layer "F.Cu") (net 42))
+  (segment (start 142.075636 115.67548) (end 145.599992 119.199836) (width 0.25) (layer "F.Cu") (net 42))
   (segment (start 120.525481 113.175325) (end 126.549992 119.199836) (width 0.25) (layer "F.Cu") (net 43))
   (segment (start 86.36 105.79) (end 93.745325 113.175325) (width 0.25) (layer "F.Cu") (net 43))

Commit message: Finilize project
Routing:
- net col1: track 19.0 -> 38.0 mm
- net col0: track 19.1 -> 29.9 mm
Changed lines of the file:
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@@
   (segment (start 117.73 102.49) (end 119.38 104.14) (width 0.25) (layer "B.Cu") (net 2))
   (segment (start 107.499992 114.299836) (end 88.449992 114.299836) (width 0.25) (layer "F.Cu") (net 3))
+  (segment (start 107.499992 114.299836) (end 107.499992 105.860008) (width 0.25) (layer "B.Cu") (net 3))
+  (segment (start 107.499992 105.860008) (end 109.22 104.14) (width 0.25) (layer "B.Cu") (net 3))
   (segment (start 126.549992 114.299836) (end 145.599992 114.299836) (width 0.25) (layer "F.Cu") (net 4))
+  (segment (start 126.549992 114.299836) (end 121.919836 114.299836) (width 0.25) (layer "B.Cu") (net 4))
+  (segment (start 121.919836 114.299836) (end 111.76 104.14) (width 0.25) (layer "B.Cu") (net 4))
   (via (at 88.9 105.918) (size 0.8) (drill 0.4) (layers "F.Cu" "B.Cu") (net 40))
   (segment (start 102.181836 119.199836) (end 107.499992 119.199836) (width 0.25) (layer "B.Cu") (net 40))
